File: RP2354-fido.kicad_pcb (KiCad board)
At the start: 2 copper layers, 28 parts, among them J1 USB_C_Receptacle_USB2.0_14P, SW1 SW_Push, U2 AP2112K-3.3, U3 USBLC6-2SC6, U4 RP2354A, Y1 Crystal

Commit message: more changes
Parts:
- removed TP1, TP2: TestPoint, TestPoint:TestPoint_Pad_1.0x1.0mm
- added J2: Conn_01x04_Pin, Connector_PinHeader_2.54mm:PinHeader_1x04_P2.54mm_Vertical, F.Cu at (196.5, 62.5)
- L1: footprint Crystal:Crystal_SMD_3225-4Pin_3.2x2.5mm -> Inductor_SMD:L_0603_1608Metric
- moved C1 49.4 mm to (105.5, 66.5)
- moved C10 47.0 mm to (113.5, 78.9)
- moved C2 47.0 mm to (110.6, 73.0)
- moved C3 47.0 mm to (110.6, 75.0)
- moved C4 47.0 mm to (110.6, 76.9)
- moved C5 47.0 mm to (110.6, 78.9)
- moved C7 47.0 mm to (113.5, 73.0)
- moved R1 43.7 mm to (141.5, 65.5), turned to 0 degrees
- moved R5 43.3 mm to (190.0, 63.5)
- moved L1 42.1 mm to (187.0, 74.0), turned to 180 degrees
- moved C9 40.2 mm to (192.5, 61.5), turned to -90 degrees
- moved D1 39.4 mm to (132.5, 75.5), turned to 0 degrees
- moved C6 39.2 mm to (119.5, 66.0)
- moved U2 39.0 mm to (132.9, 66.9)
- moved R2 37.2 mm to (141.5, 67.5), turned to 0 degrees
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Routing:
- net GND: track 18.4 -> 0.00 mm
- net (no net): track 12.3 -> 0.00 mm, vias 3 -> 0
- net Net-(J1-D+-PadA6): track 10.7 -> 0.00 mm
- net Net-(J1-D--PadA7): track 8.04 -> 0.00 mm
- net Net-(J1-CC1): track 7.97 -> 0.00 mm
- net Net-(J1-CC2): track 7.36 -> 0.00 mm
- net unconnected-(U4-QSPI_SCLK-Pad56): track 1.90 -> 0.00 mm
- net Net-(R6-Pad1): track 1.70 -> 0.00 mm
- net Net-(R7-Pad1): track 1.65 -> 0.00 mm
- removed copper zone on B.Cu, net GND
Other:
- board outline added: 18.5 x 36 mm

Commit message: power stuff
Parts:
- moved C1 72.8 mm to (169.0, 31.0)
- moved C10 72.8 mm to (177.0, 43.4)
- moved C11 72.8 mm to (200.3, 47.0)
- moved C2 72.8 mm to (174.2, 37.5)
- moved C3 72.8 mm to (174.2, 39.5)
- moved C4 72.8 mm to (174.2, 41.4)
- moved C5 72.8 mm to (174.2, 43.4)
- moved C6 72.8 mm to (183.0, 30.5)
- moved C7 72.8 mm to (177.0, 37.5)
- moved D1 72.8 mm to (196.0, 40.0)
- moved R1 59.5 mm to (196.5, 88.0)
- moved R2 59.5 mm to (196.5, 90.0)
- moved U2 49.7 mm to (182.5, 69.5), turned to 90 degrees
- moved R3 46.4 mm to (187.5, 63.5)
- moved R4 13.5 mm to (185.5, 63.5), turned to 180 degrees
